File: Mabee_DHT11 sensor/Hardware/Mabee_DHT11 sensor V1.1.brd (EAGLE design)
At the start: 20 x 40 mm, 8 parts

Commit message: change
Connections:
- net N$2 renamed NC
Changed lines of the file:
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@@
 <wire x1="11.32" y1="23.732" x2="11.32" y2="37.78" width="0.4064" layer="16"/>
 </signal>
-<signal name="N$2">
+<signal name="NC">
 <contactref element="J1" pad="2"/>
 </signal>
