File: Mabee_DHT11 sensor/Hardware/Mabee_DHT11 sensor V1.1.sch (EAGLE design)
At the start: 7 parts

Commit message: change
Connections:
- net N$2 renamed NC
Other:
- note added: "Mabee_DHT11 sensor V1.1"
- note added: "www.makerfabs.com"
Changed lines of the file:
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@@
 <wire x1="99.06" y1="60.96" x2="99.06" y2="0" width="0.1524" layer="97"/>
 <wire x1="99.06" y1="0" x2="0" y2="0" width="0.1524" layer="97"/>
+<text x="76.2" y="58.42" size="1.016" layer="97">Mabee_DHT11 sensor V1.1</text>
+<text x="76.2" y="55.88" size="1.016" layer="97">www.makerfabs.com</text>
 </plain>
 <instances>
@@
 <segment>
 <pinref part="J1" gate="G$1" pin="1"/>
-<wire x1="83.82" y1="21.59" x2="74.93" y2="21.59" width="0.1524" layer="91"/>
+<wire x1="83.82" y1="21.59" x2="80.01" y2="21.59" width="0.1524" layer="91"/>
 <label x="80.01" y="21.59" size="1.016" layer="95"/>
 </segment>
 </net>
-<net name="N$2" class="0">
+<net name="NC" class="0">
 <segment>
 <pinref part="J1" gate="G$1" pin="2"/>
-<wire x1="83.82" y1="19.05" x2="74.93" y2="19.05" width="0.1524" layer="91"/>
+<wire x1="83.82" y1="19.05" x2="80.01" y2="19.05" width="0.1524" layer="91"/>
+<label x="80.01" y="19.05" size="1.016" layer="95"/>
 </segment>
 </net>
