File: Mabee_Relay_10A/Hardware/Mabee_Relay_10A V1.1.brd (EAGLE design)
At the start: 20 x 60 mm, 10 parts, among them K1 JQC3FF

Commit message: change
Connections:
- new net NC: J1.2
Changed lines of the file:
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@@
 </polygon>
+</signal>
+<signal name="NC">
+<contactref element="J1" pad="2"/>
 </signal>
 </signals>
