File: Mabee_Relay_10A/Hardware/Mabee_Relay_10A V1.1.sch (EAGLE design)
At the start: 9 parts, among them K1 JQC3FF

Commit message: change
Connections:
- new net NC: J1.2
Other:
- note added: "Mabee_Relay_10A V1.1"
- note added: "www.makerfabs.com"
Changed lines of the file:
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@@
 <wire x1="132.08" y1="76.2" x2="132.08" y2="0" width="0.1524" layer="97"/>
 <wire x1="132.08" y1="0" x2="0" y2="0" width="0.1524" layer="97"/>
+<text x="110.49" y="72.39" size="1.016" layer="97">Mabee_Relay_10A V1.1</text>
+<text x="110.49" y="69.85" size="1.016" layer="97">www.makerfabs.com</text>
 </plain>
 <instances>
@@
 </segment>
 </net>
+<net name="NC" class="0">
+<segment>
+<pinref part="J1" gate="G$1" pin="2"/>
+<wire x1="113.03" y1="33.02" x2="109.22" y2="33.02" width="0.1524" layer="91"/>
+<label x="109.22" y="33.02" size="0.8128" layer="95" ratio="6"/>
+</segment>
+</net>
