File: Mabee_Button/Hardware/Mabee_Button V1.1.brd (EAGLE design)
At the start: 20 x 40 mm, 6 parts

Commit message: change
Connections:
- removed net N$3: BTN.2
- net OUT: no longer BTN.4
Changed lines of the file:
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@@
 </signal>
 <signal name="OUT">
-<contactref element="BTN" pad="4"/>
 <contactref element="BTN" pad="3"/>
 <contactref element="R1" pad="2"/>
@@
 <wire x1="10.6728125" y1="17.3987" x2="11.9428125" y2="18.6687" width="0.4064" layer="1"/>
 <wire x1="11.9428125" y1="18.6687" x2="12.639959375" y2="18.6687" width="0.4064" layer="1"/>
-<wire x1="12.639959375" y1="18.6687" x2="12.639959375" y2="31.1687" width="0" layer="19" extent="1-1"/>
-</signal>
-<signal name="N$3">
-<contactref element="BTN" pad="2"/>
 </signal>
 <signal name="NC">
