File: Mabee_Button/Hardware/Mabee_Button V1.1.sch (EAGLE design)
At the start: 5 parts

Commit message: change
Other:
- note added: "Mabee_Button V1.1"
- note added: "www.makerfabs.com"
Changed lines of the file:
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@@
 <wire x1="76.2" y1="66.04" x2="76.2" y2="0" width="0.1524" layer="97"/>
 <wire x1="76.2" y1="0" x2="0" y2="0" width="0.1524" layer="97"/>
+<text x="10.16" y="5.08" size="1.4224" layer="97">Mabee_Button V1.1</text>
+<text x="10.16" y="2.54" size="1.4224" layer="97">www.makerfabs.com</text>
 </plain>
 <instances>
@@
 <pinref part="J1" gate="G$1" pin="1"/>
 <wire x1="64.77" y1="19.05" x2="58.42" y2="19.05" width="0.1524" layer="91"/>
-<label x="58.42" y="19.05" size="1.27" layer="95"/>
+<label x="58.42" y="19.05" size="0.8128" layer="95"/>
 </segment>
 </net>
@@
 <pinref part="J1" gate="G$1" pin="2"/>
 <wire x1="64.77" y1="16.51" x2="58.42" y2="16.51" width="0.1524" layer="91"/>
+<label x="58.42" y="16.51" size="0.8128" layer="95"/>
 </segment>
 </net>

Commit message: change
Connections:
- removed net N$3: BTN.2
- net OUT: no longer BTN.4
Changed lines of the file:
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@@
 <setting verticaltext="up"/>
 </settings>
-<grid distance="50" unitdist="mil" unit="mil" style="lines" multiple="1" display="yes" altdistance="0.01" altunitdist="inch" altunit="inch"/>
+<grid distance="0.1" unitdist="inch" unit="inch" style="lines" multiple="1" display="no" altdistance="0.01" altunitdist="inch" altunit="inch"/>
 <layers>
 <layer number="1" name="Top" color="4" fill="1" visible="no" active="no"/>
@@
 <net name="OUT" class="0">
 <segment>
-<pinref part="BTN" gate="G$1" pin="4"/>
-<wire x1="35.56" y1="43.18" x2="38.1" y2="43.18" width="0.1524" layer="91"/>
-</segment>
-<segment>
 <pinref part="BTN" gate="G$1" pin="3"/>
 <wire x1="17.78" y1="43.18" x2="11.43" y2="43.18" width="0.1524" layer="91"/>
@@
 </segment>
 </net>
-<net name="N$3" class="0">
-<segment>
-<pinref part="BTN" gate="G$1" pin="2"/>
-<wire x1="35.56" y1="45.72" x2="38.1" y2="45.72" width="0.1524" layer="91"/>
-</segment>
-</net>
